Commit message: two joints

File: body.urdf (robot description, URDF)
Before this commit: robot robot, 2 links, 1 joints
Links:
- removed link Leg
- added link BackLeg, mass 1; collision box size=1 1 1; visual box size=1 1 1
- added link FrontLeg, mass 1; collision box size=1 1 1; visual box size=1 1 1
Joints:
- removed joint Torso_Leg
- added joint Torso_BackLeg: type revolute, parent Torso, child BackLeg, origin xyz=.5 0 1 rpy=0 0 0, axis 0 1 0, limit lower=-3.14159 upper=3.14159 effort=0.0 velocity=0.0
- added joint Torso_FrontLeg: type revolute, parent Torso, child FrontLeg, origin xyz=-.5 0 1 rpy=0 0 0, axis 0 1 0, limit lower=-3.14159 upper=3.14159 effort=0.0 velocity=0.0

Commit message: 46

File: body.urdf (robot description, URDF)
Before this commit: robot robot, 3 links, 2 joints
Links:
- added link LeftLeg, mass 1; collision box size=1 0.2 0.2; visual box size=1 0.2 0.2
- added link LowerBackLeg, mass 1; collision box size=0.2 0.2 1; visual box size=0.2 0.2 1
- added link LowerFrontLeg, mass 1; collision box size=0.2 0.2 1; visual box size=0.2 0.2 1
- added link LowerLeftLeg, mass 1; collision box size=0.2 0.2 1; visual box size=0.2 0.2 1
- added link LowerRightLeg, mass 1; collision box size=0.2 0.2 1; visual box size=0.2 0.2 1
- added link RightLeg, mass 1; collision box size=1 0.2 0.2; visual box size=1 0.2 0.2
- link BackLeg: geometry collision box size=0.2 1 0.2; visual box size=0.2 1 0.2
- link FrontLeg: geometry collision box size=0.2 1 0.2; visual box size=0.2 1 0.2
Joints:
- added joint BackLeg_LowerBackLeg: type revolute, parent BackLeg, child LowerBackLeg, origin xyz=0 -1 0 rpy=0 0 0, axis 1 0 0, limit lower=-3.14159 upper=3.14159 effort=0.0 velocity=0.0
- added joint FrontLeg_LowerFrontLeg: type revolute, parent FrontLeg, child LowerFrontLeg, origin xyz=0 1 0 rpy=0 0 0, axis 1 0 0, limit lower=-3.14159 upper=3.14159 effort=0.0 velocity=0.0
- added joint LeftLeg_LowerLeftLeg: type revolute, parent LeftLeg, child LowerLeftLeg, origin xyz=-1 0 0 rpy=0 0 0, axis 0 1 0, limit lower=-3.14159 upper=3.14159 effort=0.0 velocity=0.0
- added joint RightLeg_LowerRightLeg: type revolute, parent RightLeg, child LowerRightLeg, origin xyz=1 0 0 rpy=0 0 0, axis 0 1 0, limit lower=-3.14159 upper=3.14159 effort=0.0 velocity=0.0
- added joint Torso_LeftLeg: type revolute, parent Torso, child LeftLeg, origin xyz=-0.5 0 1 rpy=0 0 0, axis 0 1 0, limit lower=-3.14159 upper=3.14159 effort=0.0 velocity=0.0
- added joint Torso_RightLeg: type revolute, parent Torso, child RightLeg, origin xyz=0.5 0 1 rpy=0 0 0, axis 0 1 0, limit lower=-3.14159 upper=3.14159 effort=0.0 velocity=0.0
- joint Torso_BackLeg: axis 0 1 0 -> 1 0 0; origin xyz=.5 0 1 rpy=0 0 0 -> xyz=0 -0.5 1 rpy=0 0 0
- joint Torso_FrontLeg: axis 0 1 0 -> 1 0 0; origin xyz=-.5 0 1 rpy=0 0 0 -> xyz=0 0.5 1 rpy=0 0 0

Commit message: ahhh

File: body.urdf (robot description, URDF)
Before this commit: robot robot, 9 links, 8 joints
Links:
- removed link BackLeg
- removed link FrontLeg
- removed link LeftLeg
- removed link LowerBackLeg
- removed link LowerFrontLeg
- removed link LowerLeftLeg
- removed link LowerRightLeg
- removed link RightLeg
- added link LowerLeg0, mass 1; collision box size=0.2 0.2 1; visual box size=0.2 0.2 1
- added link LowerLeg1, mass 1; collision box size=0.2 0.2 1; visual box size=0.2 0.2 1
- added link LowerLeg2, mass 1; collision box size=0.2 0.2 1; visual box size=0.2 0.2 1
- added link LowerLeg3, mass 1; collision box size=0.2 0.2 1; visual box size=0.2 0.2 1
- added link UppperLeg0, mass 1; collision box size=0.2 1 0.2; visual box size=0.2 1 0.2
- added link UppperLeg1, mass 1; collision box size=0.2 1 0.2; visual box size=0.2 1 0.2
- added link UppperLeg2, mass 1; collision box size=0.2 1 0.2; visual box size=0.2 1 0.2
- added link UppperLeg3, mass 1; collision box size=0.2 1 0.2; visual box size=0.2 1 0.2
Joints:
- removed joint BackLeg_LowerBackLeg
- removed joint FrontLeg_LowerFrontLeg
- removed joint LeftLeg_LowerLeftLeg
- removed joint RightLeg_LowerRightLeg
- removed joint Torso_BackLeg
- removed joint Torso_FrontLeg
- removed joint Torso_LeftLeg
- removed joint Torso_RightLeg
- added joint Torso_UppperLeg0: type revolute, parent Torso, child Leg0, origin xyz=0.5 0 1 rpy=0 0 0, axis 0 1 0, limit lower=-3.14159 upper=3.14159 effort=0.0 velocity=0.0
- added joint Torso_UppperLeg1: type revolute, parent Torso, child Leg1, origin xyz=0 0.5 1 rpy=0 0 0, axis 0 1 0, limit lower=-3.14159 upper=3.14159 effort=0.0 velocity=0.0
- added joint Torso_UppperLeg2: type revolute, parent Torso, child Leg2, origin xyz=-0.5 0 1 rpy=0 0 0, axis 1 0 0, limit lower=-3.14159 upper=3.14159 effort=0.0 velocity=0.0
- added joint Torso_UppperLeg3: type revolute, parent Torso, child Leg3, origin xyz=0 -0.5 1 rpy=0 0 0, axis 0 1 0, limit lower=-3.14159 upper=3.14159 effort=0.0 velocity=0.0
- added joint UppperLeg0_LowerLeg0: type revolute, parent Leg0, child LowerLeg0, origin xyz=1 0 0 rpy=0 0 0, axis 0 1 0, limit lower=-3.14159 upper=3.14159 effort=0.0 velocity=0.0
- added joint UppperLeg1_LowerLeg1: type revolute, parent Leg1, child LowerLeg1, origin xyz=0 1 0 rpy=0 0 0, axis 1 0 0, limit lower=-3.14159 upper=3.14159 effort=0.0 velocity=0.0
- added joint UppperLeg2_LowerLeg2: type revolute, parent Leg2, child LowerLeg2, origin xyz=-1 0 0 rpy=0 0 0, axis 0 1 0, limit lower=-3.14159 upper=3.14159 effort=0.0 velocity=0.0
- added joint UppperLeg3_LowerLeg3: type revolute, parent Leg3, child LowerLeg3, origin xyz=-1 0 0 rpy=0 0 0, axis 0 1 0, limit lower=-3.14159 upper=3.14159 effort=0.0 velocity=0.0

Commit message: naming is hard

File: body.urdf (robot description, URDF)
Before this commit: robot robot, 9 links, 8 joints
Links:
- removed link LowerLeg1
- removed link LowerLeg2
- removed link LowerLeg3
- removed link UppperLeg1
- removed link UppperLeg2
- removed link UppperLeg3
- link UppperLeg0: geometry collision box size=1 0.2 0.2; visual box size=1 0.2 0.2
Joints:
- removed joint Torso_UppperLeg1
- removed joint Torso_UppperLeg2
- removed joint Torso_UppperLeg3
- removed joint UppperLeg1_LowerLeg1
- removed joint UppperLeg2_LowerLeg2
- removed joint UppperLeg3_LowerLeg3
- joint Torso_UppperLeg0: child Leg0 -> UppperLeg0
- joint UppperLeg0_LowerLeg0: parent Leg0 -> UppperLeg0

Commit message: sphere body

File: body.urdf (robot description, URDF)
Before this commit: robot robot, 3 links, 2 joints
Links:
- added link LowerLeg1, mass 1; collision box size=0.2 0.2 1; visual box size=0.2 0.2 1
- added link LowerLeg2, mass 1; collision box size=0.2 0.2 1; visual box size=0.2 0.2 1
- added link LowerLeg3, mass 1; collision box size=0.2 0.2 1; visual box size=0.2 0.2 1
- added link UppperLeg1, mass 1; collision box size=0.2 1 0.2; visual box size=0.2 1 0.2
- added link UppperLeg2, mass 1; collision box size=1 0.2 0.2; visual box size=1 0.2 0.2
- added link UppperLeg3, mass 1; collision box size=0.2 1 0.2; visual box size=0.2 1 0.2
- link Torso: geometry collision sphere radius=0.5; visual sphere radius=0.5
Joints:
- added joint Torso_UppperLeg1: type revolute, parent Torso, child UppperLeg1, origin xyz=0 0.5 1 rpy=0 0 0, axis 1 0 0, limit lower=-3.14159 upper=3.14159 effort=0.0 velocity=0.0
- added joint Torso_UppperLeg2: type revolute, parent Torso, child UppperLeg2, origin xyz=-0.5 0 1 rpy=0 0 0, axis 0 1 0, limit lower=-3.14159 upper=3.14159 effort=0.0 velocity=0.0
- added joint Torso_UppperLeg3: type revolute, parent Torso, child UppperLeg3, origin xyz=0 -0.5 1 rpy=0 0 0, axis 1 0 0, limit lower=-3.14159 upper=3.14159 effort=0.0 velocity=0.0
- added joint UppperLeg1_LowerLeg1: type revolute, parent UppperLeg1, child LowerLeg1, origin xyz=0 1 0 rpy=0 0 0, axis 1 0 0, limit lower=-3.14159 upper=3.14159 effort=0.0 velocity=0.0
- added joint UppperLeg2_LowerLeg2: type revolute, parent UppperLeg2, child LowerLeg2, origin xyz=-1 0 0 rpy=0 0 0, axis 0 1 0, limit lower=-3.14159 upper=3.14159 effort=0.0 velocity=0.0
- added joint UppperLeg3_LowerLeg3: type revolute, parent UppperLeg3, child LowerLeg3, origin xyz=0 -1 0 rpy=0 0 0, axis 1 0 0, limit lower=-3.14159 upper=3.14159 effort=0.0 velocity=0.0

Commit message: legs

File: body.urdf (robot description, URDF)
Before this commit: robot robot, 9 links, 8 joints
Joints:
- joint Torso_UppperLeg0: origin xyz=0.5 0 1 rpy=0 0 0 -> xyz=0.5 0.0 1 rpy=0 0 0
- joint Torso_UppperLeg1: origin xyz=0 0.5 1 rpy=0 0 0 -> xyz=3.061616997868383e-17 0.5 1 rpy=0 0 0
- joint Torso_UppperLeg2: origin xyz=-0.5 0 1 rpy=0 0 0 -> xyz=-0.5 6.123233995736766e-17 1 rpy=0 0 0
- joint Torso_UppperLeg3: origin xyz=0 -0.5 1 rpy=0 0 0 -> xyz=-9.184850993605148e-17 -0.5 1 rpy=0 0 0

Commit message: fixed motors and sensor constant

File: body.urdf (robot description, URDF)
Before this commit: robot robot, 9 links, 8 joints
Links:
- removed link LowerLeg1
- removed link LowerLeg2
- removed link LowerLeg3
- removed link UppperLeg1
- removed link UppperLeg2
- removed link UppperLeg3
Joints:
- removed joint Torso_UppperLeg1
- removed joint Torso_UppperLeg2
- removed joint Torso_UppperLeg3
- removed joint UppperLeg1_LowerLeg1
- removed joint UppperLeg2_LowerLeg2
- removed joint UppperLeg3_LowerLeg3

Commit message: mass broke

File: body.urdf (robot description, URDF)
Before this commit: robot robot, 3 links, 2 joints
Links:
- added link LowerLeg1, mass box; collision sphere radius=0.2; visual sphere radius=0.2
- added link LowerLeg2, mass box; collision sphere radius=0.2; visual sphere radius=0.2
- added link LowerLeg3, mass box; collision sphere radius=0.2; visual sphere radius=0.2
- added link UppperLeg1, mass box; collision sphere radius=0.2; visual sphere radius=0.2
- added link UppperLeg2, mass box; collision sphere radius=1; visual sphere radius=1
- added link UppperLeg3, mass box; collision sphere radius=0.2; visual sphere radius=0.2
- link LowerLeg0: mass 1 -> box; geometry collision sphere radius=0.2; visual sphere radius=0.2
- link Torso: mass 1 -> sphere
- link UppperLeg0: mass 1 -> box; geometry collision sphere radius=1; visual sphere radius=1
Joints:
- added joint Torso_UppperLeg1: type revolute, parent Torso, child UppperLeg1, origin xyz=3.061616997868383e-17 0.5 1 rpy=0 0 0, axis 1 0 0, limit lower=-3.14159 upper=3.14159 effort=0.0 velocity=0.0
- added joint Torso_UppperLeg2: type revolute, parent Torso, child UppperLeg2, origin xyz=-0.5 6.123233995736766e-17 1 rpy=0 0 0, axis 0 1 0, limit lower=-3.14159 upper=3.14159 effort=0.0 velocity=0.0
- added joint Torso_UppperLeg3: type revolute, parent Torso, child UppperLeg3, origin xyz=-9.184850993605148e-17 -0.5 1 rpy=0 0 0, axis 1 0 0, limit lower=-3.14159 upper=3.14159 effort=0.0 velocity=0.0
- added joint UppperLeg1_LowerLeg1: type revolute, parent UppperLeg1, child LowerLeg1, origin xyz=0 1 0 rpy=0 0 0, axis 1 0 0, limit lower=-3.14159 upper=3.14159 effort=0.0 velocity=0.0
- added joint UppperLeg2_LowerLeg2: type revolute, parent UppperLeg2, child LowerLeg2, origin xyz=-1 0 0 rpy=0 0 0, axis 0 1 0, limit lower=-3.14159 upper=3.14159 effort=0.0 velocity=0.0
- added joint UppperLeg3_LowerLeg3: type revolute, parent UppperLeg3, child LowerLeg3, origin xyz=0 -1 0 rpy=0 0 0, axis 1 0 0, limit lower=-3.14159 upper=3.14159 effort=0.0 velocity=0.0

Commit message: Revert "mass broke"
This reverts commit c633aec9e1b684c2e740339ab50d26118cdf490c.

File: body.urdf (robot description, URDF)
Before this commit: robot robot, 9 links, 8 joints
Links:
- removed link LowerLeg1
- removed link LowerLeg2
- removed link LowerLeg3
- removed link UppperLeg1
- removed link UppperLeg2
- removed link UppperLeg3
- link LowerLeg0: mass box -> 1; geometry collision box size=0.2 0.2 1; visual box size=0.2 0.2 1
- link Torso: mass sphere -> 1
- link UppperLeg0: mass box -> 1; geometry collision box size=1 0.2 0.2; visual box size=1 0.2 0.2
Joints:
- removed joint Torso_UppperLeg1
- removed joint Torso_UppperLeg2
- removed joint Torso_UppperLeg3
- removed joint UppperLeg1_LowerLeg1
- removed joint UppperLeg2_LowerLeg2
- removed joint UppperLeg3_LowerLeg3

Commit message: working agian

File: body.urdf (robot description, URDF)
Before this commit: robot robot, 3 links, 2 joints
Links:
- added link LowerLeg1, mass 1; collision box size=0.2 0.2 1; visual box size=0.2 0.2 1
- added link LowerLeg2, mass 1; collision box size=0.2 0.2 1; visual box size=0.2 0.2 1
- added link LowerLeg3, mass 1; collision box size=0.2 0.2 1; visual box size=0.2 0.2 1
- added link UppperLeg1, mass 1; collision box size=0.2 1 0.2; visual box size=0.2 1 0.2
- added link UppperLeg2, mass 1; collision box size=1 0.2 0.2; visual box size=1 0.2 0.2
- added link UppperLeg3, mass 1; collision box size=0.2 1 0.2; visual box size=0.2 1 0.2
Joints:
- added joint Torso_UppperLeg1: type revolute, parent Torso, child UppperLeg1, origin xyz=3.061616997868383e-17 0.5 1 rpy=0 0 0, axis 1 0 0, limit lower=-3.14159 upper=3.14159 effort=0.0 velocity=0.0
- added joint Torso_UppperLeg2: type revolute, parent Torso, child UppperLeg2, origin xyz=-0.5 6.123233995736766e-17 1 rpy=0 0 0, axis 0 1 0, limit lower=-3.14159 upper=3.14159 effort=0.0 velocity=0.0
- added joint Torso_UppperLeg3: type revolute, parent Torso, child UppperLeg3, origin xyz=-9.184850993605148e-17 -0.5 1 rpy=0 0 0, axis 1 0 0, limit lower=-3.14159 upper=3.14159 effort=0.0 velocity=0.0
- added joint UppperLeg1_LowerLeg1: type revolute, parent UppperLeg1, child LowerLeg1, origin xyz=0 1 0 rpy=0 0 0, axis 1 0 0, limit lower=-3.14159 upper=3.14159 effort=0.0 velocity=0.0
- added joint UppperLeg2_LowerLeg2: type revolute, parent UppperLeg2, child LowerLeg2, origin xyz=-1 0 0 rpy=0 0 0, axis 0 1 0, limit lower=-3.14159 upper=3.14159 effort=0.0 velocity=0.0
- added joint UppperLeg3_LowerLeg3: type revolute, parent UppperLeg3, child LowerLeg3, origin xyz=0 -1 0 rpy=0 0 0, axis 1 0 0, limit lower=-3.14159 upper=3.14159 effort=0.0 velocity=0.0

Commit message: so many legs attached correctly, not sure if

File: body.urdf (robot description, URDF)
Before this commit: robot robot, 9 links, 8 joints
Links:
- added link LowerLeg10, mass 1; collision box size=0.2 0.2 1; visual box size=0.2 0.2 1
- added link LowerLeg11, mass 1; collision box size=0.2 0.2 1; visual box size=0.2 0.2 1
- added link LowerLeg12, mass 1; collision box size=0.2 0.2 1; visual box size=0.2 0.2 1
- added link LowerLeg4, mass 1; collision box size=0.2 0.2 1; visual box size=0.2 0.2 1
- added link LowerLeg5, mass 1; collision box size=0.2 0.2 1; visual box size=0.2 0.2 1
- added link LowerLeg6, mass 1; collision box size=0.2 0.2 1; visual box size=0.2 0.2 1
- added link LowerLeg7, mass 1; collision box size=0.2 0.2 1; visual box size=0.2 0.2 1
- added link LowerLeg8, mass 1; collision box size=0.2 0.2 1; visual box size=0.2 0.2 1
- added link LowerLeg9, mass 1; collision box size=0.2 0.2 1; visual box size=0.2 0.2 1
- added link UppperLeg10, mass 1; collision box size=1 0.2 0.2; visual box size=1 0.2 0.2
- added link UppperLeg11, mass 1; collision box size=1 0.2 0.2; visual box size=1 0.2 0.2
- added link UppperLeg12, mass 1; collision box size=1 0.2 0.2; visual box size=1 0.2 0.2
- added link UppperLeg4, mass 1; collision box size=1 0.2 0.2; visual box size=1 0.2 0.2
- added link UppperLeg5, mass 1; collision box size=1 0.2 0.2; visual box size=1 0.2 0.2
- added link UppperLeg6, mass 1; collision box size=1 0.2 0.2; visual box size=1 0.2 0.2
- added link UppperLeg7, mass 1; collision box size=1 0.2 0.2; visual box size=1 0.2 0.2
- added link UppperLeg8, mass 1; collision box size=1 0.2 0.2; visual box size=1 0.2 0.2
- added link UppperLeg9, mass 1; collision box size=1 0.2 0.2; visual box size=1 0.2 0.2
- link UppperLeg1: geometry collision box size=1 0.2 0.2; visual box size=1 0.2 0.2
- link UppperLeg3: geometry collision box size=1 0.2 0.2; visual box size=1 0.2 0.2
Joints:
- added joint Torso_UppperLeg10: type revolute, parent Torso, child UppperLeg10, origin xyz=0.06026834012766116 -0.49635443704902704 1 rpy=0 0 0, axis 0.06026834012766116 -0.49635443704902704 0, limit lower=-3.14159 upper=3.14159 effort=0.0 velocity=0.0
- added joint Torso_UppperLeg11: type revolute, parent Torso, child UppperLeg11, origin xyz=0.28403237336557813 -0.411491932946828 1 rpy=0 0 0, axis 0.28403237336557813 -0.411491932946828 0, limit lower=-3.14159 upper=3.14159 effort=0.0 velocity=0.0
- added joint Torso_UppperLeg12: type revolute, parent Torso, child UppperLeg12, origin xyz=0.442728012826605 -0.2323615860218842 1 rpy=0 0 0, axis 0.442728012826605 -0.2323615860218842 0, limit lower=-3.14159 upper=3.14159 effort=0.0 velocity=0.0
- added joint Torso_UppperLeg4: type revolute, parent Torso, child UppperLeg4, origin xyz=-0.17730244352126784 0.4675081213427074 1 rpy=0 0 0, axis -0.17730244352126784 0.4675081213427074 0, limit lower=-3.14159 upper=3.14159 effort=0.0 velocity=0.0
- added joint Torso_UppperLeg5: type revolute, parent Torso, child UppperLeg5, origin xyz=-0.37425537408555043 0.3315613291203977 1 rpy=0 0 0, axis -0.37425537408555043 0.3315613291203977 0, limit lower=-3.14159 upper=3.14159 effort=0.0 velocity=0.0
- added joint Torso_UppperLeg6: type revolute, parent Torso, child UppperLeg6, origin xyz=-0.485470908713026 0.11965783214377884 1 rpy=0 0 0, axis -0.485470908713026 0.11965783214377884 0, limit lower=-3.14159 upper=3.14159 effort=0.0 velocity=0.0
- added joint Torso_UppperLeg7: type revolute, parent Torso, child UppperLeg7, origin xyz=-0.485470908713026 -0.11965783214377894 1 rpy=0 0 0, axis -0.485470908713026 -0.11965783214377894 0, limit lower=-3.14159 upper=3.14159 effort=0.0 velocity=0.0
- added joint Torso_UppperLeg8: type revolute, parent Torso, child UppperLeg8, origin xyz=-0.3742553740855505 -0.33156132912039765 1 rpy=0 0 0, axis -0.3742553740855505 -0.33156132912039765 0, limit lower=-3.14159 upper=3.14159 effort=0.0 velocity=0.0
- added joint Torso_UppperLeg9: type revolute, parent Torso, child UppperLeg9, origin xyz=-0.17730244352126795 -0.46750812134270736 1 rpy=0 0 0, axis -0.17730244352126795 -0.46750812134270736 0, limit lower=-3.14159 upper=3.14159 effort=0.0 velocity=0.0
- added joint UppperLeg10_LowerLeg10: type revolute, parent UppperLeg10, child LowerLeg10, origin xyz=0.12053668025532233 -0.9927088740980541 0 rpy=0 0 0, axis 0.06026834012766116 -0.49635443704902704 0, limit lower=-3.14159 upper=3.14159 effort=0.0 velocity=0.0
- added joint UppperLeg11_LowerLeg11: type revolute, parent UppperLeg11, child LowerLeg11, origin xyz=0.5680647467311563 -0.822983865893656 0 rpy=0 0 0, axis 0.28403237336557813 -0.411491932946828 0, limit lower=-3.14159 upper=3.14159 effort=0.0 velocity=0.0
- added joint UppperLeg12_LowerLeg12: type revolute, parent UppperLeg12, child LowerLeg12, origin xyz=0.88545602565321 -0.4647231720437684 0 rpy=0 0 0, axis 0.442728012826605 -0.2323615860218842 0, limit lower=-3.14159 upper=3.14159 effort=0.0 velocity=0.0
- added joint UppperLeg4_LowerLeg4: type revolute, parent UppperLeg4, child LowerLeg4, origin xyz=-0.3546048870425357 0.9350162426854148 0 rpy=0 0 0, axis -0.17730244352126784 0.4675081213427074 0, limit lower=-3.14159 upper=3.14159 effort=0.0 velocity=0.0
- added joint UppperLeg5_LowerLeg5: type revolute, parent UppperLeg5, child LowerLeg5, origin xyz=-0.7485107481711009 0.6631226582407954 0 rpy=0 0 0, axis -0.37425537408555043 0.3315613291203977 0, limit lower=-3.14159 upper=3.14159 effort=0.0 velocity=0.0
- added joint UppperLeg6_LowerLeg6: type revolute, parent UppperLeg6, child LowerLeg6, origin xyz=-0.970941817426052 0.23931566428755768 0 rpy=0 0 0, axis -0.485470908713026 0.11965783214377884 0, limit lower=-3.14159 upper=3.14159 effort=0.0 velocity=0.0
- added joint UppperLeg7_LowerLeg7: type revolute, parent UppperLeg7, child LowerLeg7, origin xyz=-0.970941817426052 -0.23931566428755788 0 rpy=0 0 0, axis -0.485470908713026 -0.11965783214377894 0, limit lower=-3.14159 upper=3.14159 effort=0.0 velocity=0.0
- added joint UppperLeg8_LowerLeg8: type revolute, parent UppperLeg8, child LowerLeg8, origin xyz=-0.748510748171101 -0.6631226582407953 0 rpy=0 0 0, axis -0.3742553740855505 -0.33156132912039765 0, limit lower=-3.14159 upper=3.14159 effort=0.0 velocity=0.0
- added joint UppperLeg9_LowerLeg9: type revolute, parent UppperLeg9, child LowerLeg9, origin xyz=-0.3546048870425359 -0.9350162426854147 0 rpy=0 0 0, axis -0.17730244352126795 -0.46750812134270736 0, limit lower=-3.14159 upper=3.14159 effort=0.0 velocity=0.0
- joint Torso_UppperLeg0: axis 0 1 0 -> 0.5 0.0 0
- joint Torso_UppperLeg1: axis 1 0 0 -> 0.44272801282660496 0.23236158602188428 0; origin xyz=3.061616997868383e-17 0.5 1 rpy=0 0 0 -> xyz=0.44272801282660496 0.23236158602188428 1 rpy=0 0 0
- joint Torso_UppperLeg2: axis 0 1 0 -> 0.2840323733655779 0.41149193294682823 0; origin xyz=-0.5 6.123233995736766e-17 1 rpy=0 0 0 -> xyz=0.2840323733655779 0.41149193294682823 1 rpy=0 0 0
- joint Torso_UppperLeg3: axis 1 0 0 -> 0.0602683401276615 0.496354437049027 0; origin xyz=-9.184850993605148e-17 -0.5 1 rpy=0 0 0 -> xyz=0.0602683401276615 0.496354437049027 1 rpy=0 0 0
- joint UppperLeg0_LowerLeg0: axis 0 1 0 -> 0.5 0.0 0; origin xyz=1 0 0 rpy=0 0 0 -> xyz=1.0 0.0 0 rpy=0 0 0
- joint UppperLeg1_LowerLeg1: axis 1 0 0 -> 0.44272801282660496 0.23236158602188428 0; origin xyz=0 1 0 rpy=0 0 0 -> xyz=0.8854560256532099 0.46472317204376856 0 rpy=0 0 0
- joint UppperLeg2_LowerLeg2: axis 0 1 0 -> 0.2840323733655779 0.41149193294682823 0; origin xyz=-1 0 0 rpy=0 0 0 -> xyz=0.5680647467311558 0.8229838658936565 0 rpy=0 0 0
- joint UppperLeg3_LowerLeg3: axis 1 0 0 -> 0.0602683401276615 0.496354437049027 0; origin xyz=0 -1 0 rpy=0 0 0 -> xyz=0.120536680255323 0.992708874098054 0 rpy=0 0 0
