Commit message: deliverable 2

File: body.urdf (robot description, URDF)
Before this commit: robot robot, 27 links, 26 joints
Links:
- removed link LowerLeg10
- removed link LowerLeg11
- removed link LowerLeg12
- removed link LowerLeg5
- removed link LowerLeg6
- removed link LowerLeg7
- removed link LowerLeg8
- removed link LowerLeg9
- removed link UppperLeg10
- removed link UppperLeg11
- removed link UppperLeg12
- removed link UppperLeg5
- removed link UppperLeg6
- removed link UppperLeg7
- removed link UppperLeg8
- removed link UppperLeg9
Joints:
- removed joint Torso_UppperLeg10
- removed joint Torso_UppperLeg11
- removed joint Torso_UppperLeg12
- removed joint Torso_UppperLeg5
- removed joint Torso_UppperLeg6
- removed joint Torso_UppperLeg7
- removed joint Torso_UppperLeg8
- removed joint Torso_UppperLeg9
- removed joint UppperLeg10_LowerLeg10
- removed joint UppperLeg11_LowerLeg11
- removed joint UppperLeg12_LowerLeg12
- removed joint UppperLeg5_LowerLeg5
- removed joint UppperLeg6_LowerLeg6
- removed joint UppperLeg7_LowerLeg7
- removed joint UppperLeg8_LowerLeg8
- removed joint UppperLeg9_LowerLeg9
- joint Torso_UppperLeg0: axis 0.5 0.0 0 -> 0.0 1.0 0
- joint Torso_UppperLeg1: axis 0.44272801282660496 0.23236158602188428 0 -> 0.9510565162951535 0.30901699437494745 0; origin xyz=0.44272801282660496 0.23236158602188428 1 rpy=0 0 0 -> xyz=0.15450849718747373 0.47552825814757677 1 rpy=0 0 0
- joint Torso_UppperLeg2: axis 0.2840323733655779 0.41149193294682823 0 -> 0.5877852522924732 0.8090169943749473 0; origin xyz=0.2840323733655779 0.41149193294682823 1 rpy=0 0 0 -> xyz=-0.40450849718747367 0.2938926261462366 1 rpy=0 0 0
- joint Torso_UppperLeg3: axis 0.0602683401276615 0.496354437049027 0 -> 0.587785252292473 0.8090169943749475 0; origin xyz=0.0602683401276615 0.496354437049027 1 rpy=0 0 0 -> xyz=-0.4045084971874737 -0.2938926261462365 1 rpy=0 0 0
- joint Torso_UppperLeg4: axis -0.17730244352126784 0.4675081213427074 0 -> 0.9510565162951536 0.30901699437494723 0; origin xyz=-0.17730244352126784 0.4675081213427074 1 rpy=0 0 0 -> xyz=0.15450849718747361 -0.4755282581475768 1 rpy=0 0 0
- joint UppperLeg0_LowerLeg0: axis 0.5 0.0 0 -> 0.0 1.0 0
- joint UppperLeg1_LowerLeg1: axis 0.44272801282660496 0.23236158602188428 0 -> 0.9510565162951535 0.30901699437494745 0; origin xyz=0.8854560256532099 0.46472317204376856 0 rpy=0 0 0 -> xyz=0.30901699437494745 0.9510565162951535 0 rpy=0 0 0
- joint UppperLeg2_LowerLeg2: axis 0.2840323733655779 0.41149193294682823 0 -> 0.5877852522924732 0.8090169943749473 0; origin xyz=0.5680647467311558 0.8229838658936565 0 rpy=0 0 0 -> xyz=-0.8090169943749473 0.5877852522924732 0 rpy=0 0 0
- joint UppperLeg3_LowerLeg3: axis 0.0602683401276615 0.496354437049027 0 -> 0.587785252292473 0.8090169943749475 0; origin xyz=0.120536680255323 0.992708874098054 0 rpy=0 0 0 -> xyz=-0.8090169943749475 -0.587785252292473 0 rpy=0 0 0
- joint UppperLeg4_LowerLeg4: axis -0.17730244352126784 0.4675081213427074 0 -> 0.9510565162951536 0.30901699437494723 0; origin xyz=-0.3546048870425357 0.9350162426854148 0 rpy=0 0 0 -> xyz=0.30901699437494723 -0.9510565162951536 0 rpy=0 0 0

Commit message: num legs

File: body.urdf (robot description, URDF)
Before this commit: robot robot, 11 links, 10 joints
Links:
- added link LowerLeg10, mass 1; collision box size=0.2 0.2 1; visual box size=0.2 0.2 1
- added link LowerLeg11, mass 1; collision box size=0.2 0.2 1; visual box size=0.2 0.2 1
- added link LowerLeg12, mass 1; collision box size=0.2 0.2 1; visual box size=0.2 0.2 1
- added link LowerLeg13, mass 1; collision box size=0.2 0.2 1; visual box size=0.2 0.2 1
- added link LowerLeg14, mass 1; collision box size=0.2 0.2 1; visual box size=0.2 0.2 1
- added link LowerLeg5, mass 1; collision box size=0.2 0.2 1; visual box size=0.2 0.2 1
- added link LowerLeg6, mass 1; collision box size=0.2 0.2 1; visual box size=0.2 0.2 1
- added link LowerLeg7, mass 1; collision box size=0.2 0.2 1; visual box size=0.2 0.2 1
- added link LowerLeg8, mass 1; collision box size=0.2 0.2 1; visual box size=0.2 0.2 1
- added link LowerLeg9, mass 1; collision box size=0.2 0.2 1; visual box size=0.2 0.2 1
- added link UppperLeg10, mass 1; collision box size=1 0.2 0.2; visual box size=1 0.2 0.2
- added link UppperLeg11, mass 1; collision box size=1 0.2 0.2; visual box size=1 0.2 0.2
- added link UppperLeg12, mass 1; collision box size=1 0.2 0.2; visual box size=1 0.2 0.2
- added link UppperLeg13, mass 1; collision box size=1 0.2 0.2; visual box size=1 0.2 0.2
- added link UppperLeg14, mass 1; collision box size=1 0.2 0.2; visual box size=1 0.2 0.2
- added link UppperLeg5, mass 1; collision box size=1 0.2 0.2; visual box size=1 0.2 0.2
- added link UppperLeg6, mass 1; collision box size=1 0.2 0.2; visual box size=1 0.2 0.2
- added link UppperLeg7, mass 1; collision box size=1 0.2 0.2; visual box size=1 0.2 0.2
- added link UppperLeg8, mass 1; collision box size=1 0.2 0.2; visual box size=1 0.2 0.2
- added link UppperLeg9, mass 1; collision box size=1 0.2 0.2; visual box size=1 0.2 0.2
Joints:
- added joint Torso_UppperLeg10: type revolute, parent Torso, child UppperLeg10, origin xyz=-0.2500000000000002 -0.43301270189221924 1 rpy=0 0 0, axis 0.8660254037844385 0.5000000000000004 0, limit lower=-3.14159 upper=3.14159 effort=0.0 velocity=0.0
- added joint Torso_UppperLeg11: type revolute, parent Torso, child UppperLeg11, origin xyz=-0.05226423163382668 -0.4972609476841367 1 rpy=0 0 0, axis 0.9945218953682734 0.10452846326765336 0, limit lower=-3.14159 upper=3.14159 effort=0.0 velocity=0.0
- added joint Torso_UppperLeg12: type revolute, parent Torso, child UppperLeg12, origin xyz=0.15450849718747361 -0.4755282581475768 1 rpy=0 0 0, axis 0.9510565162951536 0.30901699437494723 0, limit lower=-3.14159 upper=3.14159 effort=0.0 velocity=0.0
- added joint Torso_UppperLeg13: type revolute, parent Torso, child UppperLeg13, origin xyz=0.3345653031794289 -0.3715724127386973 1 rpy=0 0 0, axis 0.7431448254773946 0.6691306063588578 0, limit lower=-3.14159 upper=3.14159 effort=0.0 velocity=0.0
- added joint Torso_UppperLeg14: type revolute, parent Torso, child UppperLeg14, origin xyz=0.4567727288213005 -0.20336832153790008 1 rpy=0 0 0, axis 0.40673664307580015 0.913545457642601 0, limit lower=-3.14159 upper=3.14159 effort=0.0 velocity=0.0
- added joint Torso_UppperLeg5: type revolute, parent Torso, child UppperLeg5, origin xyz=-0.2499999999999999 0.43301270189221935 1 rpy=0 0 0, axis 0.8660254037844387 0.4999999999999998 0, limit lower=-3.14159 upper=3.14159 effort=0.0 velocity=0.0
- added joint Torso_UppperLeg6: type revolute, parent Torso, child UppperLeg6, origin xyz=-0.40450849718747367 0.2938926261462366 1 rpy=0 0 0, axis 0.5877852522924732 0.8090169943749473 0, limit lower=-3.14159 upper=3.14159 effort=0.0 velocity=0.0
- added joint Torso_UppperLeg7: type revolute, parent Torso, child UppperLeg7, origin xyz=-0.48907380036690284 0.10395584540887966 1 rpy=0 0 0, axis 0.20791169081775931 0.9781476007338057 0, limit lower=-3.14159 upper=3.14159 effort=0.0 velocity=0.0
- added joint Torso_UppperLeg8: type revolute, parent Torso, child UppperLeg8, origin xyz=-0.4890738003669028 -0.10395584540887975 1 rpy=0 0 0, axis 0.2079116908177595 0.9781476007338056 0, limit lower=-3.14159 upper=3.14159 effort=0.0 velocity=0.0
- added joint Torso_UppperLeg9: type revolute, parent Torso, child UppperLeg9, origin xyz=-0.4045084971874737 -0.2938926261462365 1 rpy=0 0 0, axis 0.587785252292473 0.8090169943749475 0, limit lower=-3.14159 upper=3.14159 effort=0.0 velocity=0.0
- added joint UppperLeg10_LowerLeg10: type revolute, parent UppperLeg10, child LowerLeg10, origin xyz=-0.5000000000000004 -0.8660254037844385 0 rpy=0 0 0, axis 0.8660254037844385 0.5000000000000004 0, limit lower=-3.14159 upper=3.14159 effort=0.0 velocity=0.0
- added joint UppperLeg11_LowerLeg11: type revolute, parent UppperLeg11, child LowerLeg11, origin xyz=-0.10452846326765336 -0.9945218953682734 0 rpy=0 0 0, axis 0.9945218953682734 0.10452846326765336 0, limit lower=-3.14159 upper=3.14159 effort=0.0 velocity=0.0
- added joint UppperLeg12_LowerLeg12: type revolute, parent UppperLeg12, child LowerLeg12, origin xyz=0.30901699437494723 -0.9510565162951536 0 rpy=0 0 0, axis 0.9510565162951536 0.30901699437494723 0, limit lower=-3.14159 upper=3.14159 effort=0.0 velocity=0.0
- added joint UppperLeg13_LowerLeg13: type revolute, parent UppperLeg13, child LowerLeg13, origin xyz=0.6691306063588578 -0.7431448254773946 0 rpy=0 0 0, axis 0.7431448254773946 0.6691306063588578 0, limit lower=-3.14159 upper=3.14159 effort=0.0 velocity=0.0
- added joint UppperLeg14_LowerLeg14: type revolute, parent UppperLeg14, child LowerLeg14, origin xyz=0.913545457642601 -0.40673664307580015 0 rpy=0 0 0, axis 0.40673664307580015 0.913545457642601 0, limit lower=-3.14159 upper=3.14159 effort=0.0 velocity=0.0
- added joint UppperLeg5_LowerLeg5: type revolute, parent UppperLeg5, child LowerLeg5, origin xyz=-0.4999999999999998 0.8660254037844387 0 rpy=0 0 0, axis 0.8660254037844387 0.4999999999999998 0, limit lower=-3.14159 upper=3.14159 effort=0.0 velocity=0.0
- added joint UppperLeg6_LowerLeg6: type revolute, parent UppperLeg6, child LowerLeg6, origin xyz=-0.8090169943749473 0.5877852522924732 0 rpy=0 0 0, axis 0.5877852522924732 0.8090169943749473 0, limit lower=-3.14159 upper=3.14159 effort=0.0 velocity=0.0
- added joint UppperLeg7_LowerLeg7: type revolute, parent UppperLeg7, child LowerLeg7, origin xyz=-0.9781476007338057 0.20791169081775931 0 rpy=0 0 0, axis 0.20791169081775931 0.9781476007338057 0, limit lower=-3.14159 upper=3.14159 effort=0.0 velocity=0.0
- added joint UppperLeg8_LowerLeg8: type revolute, parent UppperLeg8, child LowerLeg8, origin xyz=-0.9781476007338056 -0.2079116908177595 0 rpy=0 0 0, axis 0.2079116908177595 0.9781476007338056 0, limit lower=-3.14159 upper=3.14159 effort=0.0 velocity=0.0
- added joint UppperLeg9_LowerLeg9: type revolute, parent UppperLeg9, child LowerLeg9, origin xyz=-0.8090169943749475 -0.587785252292473 0 rpy=0 0 0, axis 0.587785252292473 0.8090169943749475 0, limit lower=-3.14159 upper=3.14159 effort=0.0 velocity=0.0
- joint Torso_UppperLeg1: axis 0.9510565162951535 0.30901699437494745 0 -> 0.4067366430758002 0.9135454576426009 0; origin xyz=0.15450849718747373 0.47552825814757677 1 rpy=0 0 0 -> xyz=0.45677272882130043 0.2033683215379001 1 rpy=0 0 0
- joint Torso_UppperLeg2: axis 0.5877852522924732 0.8090169943749473 0 -> 0.7431448254773942 0.6691306063588582 0; origin xyz=-0.40450849718747367 0.2938926261462366 1 rpy=0 0 0 -> xyz=0.3345653031794291 0.3715724127386971 1 rpy=0 0 0
- joint Torso_UppperLeg3: axis 0.587785252292473 0.8090169943749475 0 -> 0.9510565162951535 0.30901699437494745 0; origin xyz=-0.4045084971874737 -0.2938926261462365 1 rpy=0 0 0 -> xyz=0.15450849718747373 0.47552825814757677 1 rpy=0 0 0
- joint Torso_UppperLeg4: axis 0.9510565162951536 0.30901699437494723 0 -> 0.9945218953682733 0.10452846326765355 0; origin xyz=0.15450849718747361 -0.4755282581475768 1 rpy=0 0 0 -> xyz=-0.05226423163382678 0.49726094768413664 1 rpy=0 0 0
- joint UppperLeg1_LowerLeg1: axis 0.9510565162951535 0.30901699437494745 0 -> 0.4067366430758002 0.9135454576426009 0; origin xyz=0.30901699437494745 0.9510565162951535 0 rpy=0 0 0 -> xyz=0.9135454576426009 0.4067366430758002 0 rpy=0 0 0
- joint UppperLeg2_LowerLeg2: axis 0.5877852522924732 0.8090169943749473 0 -> 0.7431448254773942 0.6691306063588582 0; origin xyz=-0.8090169943749473 0.5877852522924732 0 rpy=0 0 0 -> xyz=0.6691306063588582 0.7431448254773942 0 rpy=0 0 0
- joint UppperLeg3_LowerLeg3: axis 0.587785252292473 0.8090169943749475 0 -> 0.9510565162951535 0.30901699437494745 0; origin xyz=-0.8090169943749475 -0.587785252292473 0 rpy=0 0 0 -> xyz=0.30901699437494745 0.9510565162951535 0 rpy=0 0 0
- joint UppperLeg4_LowerLeg4: axis 0.9510565162951536 0.30901699437494723 0 -> 0.9945218953682733 0.10452846326765355 0; origin xyz=0.30901699437494723 -0.9510565162951536 0 rpy=0 0 0 -> xyz=-0.10452846326765355 0.9945218953682733 0 rpy=0 0 0

Commit message: robo man

File: body.urdf (robot description, URDF)
Before this commit: robot robot, 31 links, 30 joints
Links:
- removed link LowerLeg10
- removed link LowerLeg11
- removed link LowerLeg12
- removed link LowerLeg13
- removed link LowerLeg14
- removed link LowerLeg3
- removed link LowerLeg4
- removed link LowerLeg5
- removed link LowerLeg6
- removed link LowerLeg7
- removed link LowerLeg8
- removed link LowerLeg9
- removed link UppperLeg10
- removed link UppperLeg11
- removed link UppperLeg12
- removed link UppperLeg13
- removed link UppperLeg14
- removed link UppperLeg3
- removed link UppperLeg4
- removed link UppperLeg5
- removed link UppperLeg6
- removed link UppperLeg7
- removed link UppperLeg8
- removed link UppperLeg9
Joints:
- removed joint Torso_UppperLeg10
- removed joint Torso_UppperLeg11
- removed joint Torso_UppperLeg12
- removed joint Torso_UppperLeg13
- removed joint Torso_UppperLeg14
- removed joint Torso_UppperLeg3
- removed joint Torso_UppperLeg4
- removed joint Torso_UppperLeg5
- removed joint Torso_UppperLeg6
- removed joint Torso_UppperLeg7
- removed joint Torso_UppperLeg8
- removed joint Torso_UppperLeg9
- removed joint UppperLeg10_LowerLeg10
- removed joint UppperLeg11_LowerLeg11
- removed joint UppperLeg12_LowerLeg12
- removed joint UppperLeg13_LowerLeg13
- removed joint UppperLeg14_LowerLeg14
- removed joint UppperLeg3_LowerLeg3
- removed joint UppperLeg4_LowerLeg4
- removed joint UppperLeg5_LowerLeg5
- removed joint UppperLeg6_LowerLeg6
- removed joint UppperLeg7_LowerLeg7
- removed joint UppperLeg8_LowerLeg8
- removed joint UppperLeg9_LowerLeg9
- joint Torso_UppperLeg1: axis 0.4067366430758002 0.9135454576426009 0 -> 0.8660254037844387 0.4999999999999998 0; origin xyz=0.45677272882130043 0.2033683215379001 1 rpy=0 0 0 -> xyz=-0.2499999999999999 0.43301270189221935 1 rpy=0 0 0
- joint Torso_UppperLeg2: axis 0.7431448254773942 0.6691306063588582 0 -> 0.8660254037844385 0.5000000000000004 0; origin xyz=0.3345653031794291 0.3715724127386971 1 rpy=0 0 0 -> xyz=-0.2500000000000002 -0.43301270189221924 1 rpy=0 0 0
- joint UppperLeg1_LowerLeg1: axis 0.4067366430758002 0.9135454576426009 0 -> 0.8660254037844387 0.4999999999999998 0; origin xyz=0.9135454576426009 0.4067366430758002 0 rpy=0 0 0 -> xyz=-0.4999999999999998 0.8660254037844387 0 rpy=0 0 0
- joint UppperLeg2_LowerLeg2: axis 0.7431448254773942 0.6691306063588582 0 -> 0.8660254037844385 0.5000000000000004 0; origin xyz=0.6691306063588582 0.7431448254773942 0 rpy=0 0 0 -> xyz=-0.5000000000000004 -0.8660254037844385 0 rpy=0 0 0

Commit message: test walking

File: body.urdf (robot description, URDF)
Before this commit: robot robot, 7 links, 6 joints
Links:
- added link LowerLeg3, mass 1; collision box size=0.2 0.2 1; visual box size=0.2 0.2 1
- added link UppperLeg3, mass 1; collision box size=1 0.2 0.2; visual box size=1 0.2 0.2
Joints:
- added joint Torso_UppperLeg3: type revolute, parent Torso, child UppperLeg3, origin xyz=-9.184850993605148e-17 -0.5 1 rpy=0 0 0, axis 1.0 1.8369701987210297e-16 0, limit lower=-3.14159 upper=3.14159 effort=0.0 velocity=0.0
- added joint UppperLeg3_LowerLeg3: type revolute, parent UppperLeg3, child LowerLeg3, origin xyz=-1.8369701987210297e-16 -1.0 0 rpy=0 0 0, axis 1.0 1.8369701987210297e-16 0, limit lower=-3.14159 upper=3.14159 effort=0.0 velocity=0.0
- joint Torso_UppperLeg1: axis 0.8660254037844387 0.4999999999999998 0 -> 1.0 6.123233995736766e-17 0; origin xyz=-0.2499999999999999 0.43301270189221935 1 rpy=0 0 0 -> xyz=3.061616997868383e-17 0.5 1 rpy=0 0 0
- joint Torso_UppperLeg2: axis 0.8660254037844385 0.5000000000000004 0 -> 1.2246467991473532e-16 1.0 0; origin xyz=-0.2500000000000002 -0.43301270189221924 1 rpy=0 0 0 -> xyz=-0.5 6.123233995736766e-17 1 rpy=0 0 0
- joint UppperLeg1_LowerLeg1: axis 0.8660254037844387 0.4999999999999998 0 -> 1.0 6.123233995736766e-17 0; origin xyz=-0.4999999999999998 0.8660254037844387 0 rpy=0 0 0 -> xyz=6.123233995736766e-17 1.0 0 rpy=0 0 0
- joint UppperLeg2_LowerLeg2: axis 0.8660254037844385 0.5000000000000004 0 -> 1.2246467991473532e-16 1.0 0; origin xyz=-0.5000000000000004 -0.8660254037844385 0 rpy=0 0 0 -> xyz=-1.0 1.2246467991473532e-16 0 rpy=0 0 0

Commit message: idk

File: body.urdf (robot description, URDF)
Before this commit: robot robot, 9 links, 8 joints
Links:
- removed link LowerLeg3
- removed link UppperLeg3
Joints:
- removed joint Torso_UppperLeg3
- removed joint UppperLeg3_LowerLeg3
- joint Torso_UppperLeg1: axis 1.0 6.123233995736766e-17 0 -> 0.8660254037844387 0.4999999999999998 0; origin xyz=3.061616997868383e-17 0.5 1 rpy=0 0 0 -> xyz=-0.2499999999999999 0.43301270189221935 1 rpy=0 0 0
- joint Torso_UppperLeg2: axis 1.2246467991473532e-16 1.0 0 -> 0.8660254037844385 0.5000000000000004 0; origin xyz=-0.5 6.123233995736766e-17 1 rpy=0 0 0 -> xyz=-0.2500000000000002 -0.43301270189221924 1 rpy=0 0 0
- joint UppperLeg1_LowerLeg1: axis 1.0 6.123233995736766e-17 0 -> 0.8660254037844387 0.4999999999999998 0; origin xyz=6.123233995736766e-17 1.0 0 rpy=0 0 0 -> xyz=-0.4999999999999998 0.8660254037844387 0 rpy=0 0 0
- joint UppperLeg2_LowerLeg2: axis 1.2246467991473532e-16 1.0 0 -> 0.8660254037844385 0.5000000000000004 0; origin xyz=-1.0 1.2246467991473532e-16 0 rpy=0 0 0 -> xyz=-0.5000000000000004 -0.8660254037844385 0 rpy=0 0 0
