Commit message: so many legs

File: body.urdf (robot description, URDF)
Before this commit: robot robot, 9 links, 8 joints
Links:
- added link LowerLeg10, mass 1; collision box size=0.2 0.2 1; visual box size=0.2 0.2 1
- added link LowerLeg11, mass 1; collision box size=0.2 0.2 1; visual box size=0.2 0.2 1
- added link LowerLeg12, mass 1; collision box size=0.2 0.2 1; visual box size=0.2 0.2 1
- added link LowerLeg13, mass 1; collision box size=0.2 0.2 1; visual box size=0.2 0.2 1
- added link LowerLeg14, mass 1; collision box size=0.2 0.2 1; visual box size=0.2 0.2 1
- added link LowerLeg15, mass 1; collision box size=0.2 0.2 1; visual box size=0.2 0.2 1
- added link LowerLeg16, mass 1; collision box size=0.2 0.2 1; visual box size=0.2 0.2 1
- added link LowerLeg17, mass 1; collision box size=0.2 0.2 1; visual box size=0.2 0.2 1
- added link LowerLeg18, mass 1; collision box size=0.2 0.2 1; visual box size=0.2 0.2 1
- added link LowerLeg19, mass 1; collision box size=0.2 0.2 1; visual box size=0.2 0.2 1
- added link LowerLeg20, mass 1; collision box size=0.2 0.2 1; visual box size=0.2 0.2 1
- added link LowerLeg21, mass 1; collision box size=0.2 0.2 1; visual box size=0.2 0.2 1
- added link LowerLeg22, mass 1; collision box size=0.2 0.2 1; visual box size=0.2 0.2 1
- added link LowerLeg23, mass 1; collision box size=0.2 0.2 1; visual box size=0.2 0.2 1
- added link LowerLeg24, mass 1; collision box size=0.2 0.2 1; visual box size=0.2 0.2 1
- added link LowerLeg4, mass 1; collision box size=0.2 0.2 1; visual box size=0.2 0.2 1
- added link LowerLeg5, mass 1; collision box size=0.2 0.2 1; visual box size=0.2 0.2 1
- added link LowerLeg6, mass 1; collision box size=0.2 0.2 1; visual box size=0.2 0.2 1
- added link LowerLeg7, mass 1; collision box size=0.2 0.2 1; visual box size=0.2 0.2 1
- added link LowerLeg8, mass 1; collision box size=0.2 0.2 1; visual box size=0.2 0.2 1
- added link LowerLeg9, mass 1; collision box size=0.2 0.2 1; visual box size=0.2 0.2 1
- added link UppperLeg10, mass 1; collision box size=1 0.2 0.2; visual box size=1 0.2 0.2
- added link UppperLeg11, mass 1; collision box size=1 0.2 0.2; visual box size=1 0.2 0.2
- added link UppperLeg12, mass 1; collision box size=1 0.2 0.2; visual box size=1 0.2 0.2
- added link UppperLeg13, mass 1; collision box size=1 0.2 0.2; visual box size=1 0.2 0.2
- added link UppperLeg14, mass 1; collision box size=1 0.2 0.2; visual box size=1 0.2 0.2
- added link UppperLeg15, mass 1; collision box size=1 0.2 0.2; visual box size=1 0.2 0.2
- added link UppperLeg16, mass 1; collision box size=1 0.2 0.2; visual box size=1 0.2 0.2
- added link UppperLeg17, mass 1; collision box size=1 0.2 0.2; visual box size=1 0.2 0.2
- added link UppperLeg18, mass 1; collision box size=1 0.2 0.2; visual box size=1 0.2 0.2
- added link UppperLeg19, mass 1; collision box size=1 0.2 0.2; visual box size=1 0.2 0.2
- added link UppperLeg20, mass 1; collision box size=1 0.2 0.2; visual box size=1 0.2 0.2
- added link UppperLeg21, mass 1; collision box size=1 0.2 0.2; visual box size=1 0.2 0.2
- added link UppperLeg22, mass 1; collision box size=1 0.2 0.2; visual box size=1 0.2 0.2
- added link UppperLeg23, mass 1; collision box size=1 0.2 0.2; visual box size=1 0.2 0.2
- added link UppperLeg24, mass 1; collision box size=1 0.2 0.2; visual box size=1 0.2 0.2
- added link UppperLeg4, mass 1; collision box size=1 0.2 0.2; visual box size=1 0.2 0.2
- added link UppperLeg5, mass 1; collision box size=1 0.2 0.2; visual box size=1 0.2 0.2
- added link UppperLeg6, mass 1; collision box size=1 0.2 0.2; visual box size=1 0.2 0.2
- added link UppperLeg7, mass 1; collision box size=1 0.2 0.2; visual box size=1 0.2 0.2
- added link UppperLeg8, mass 1; collision box size=1 0.2 0.2; visual box size=1 0.2 0.2
- added link UppperLeg9, mass 1; collision box size=1 0.2 0.2; visual box size=1 0.2 0.2
Joints:
- added joint Torso_UppperLeg10: type revolute, parent Torso, child UppperLeg10, origin xyz=-0.40450849718747367 0.2938926261462366 1 rpy=0 0 0, axis 0.5877852522924732 0.8090169943749473 0, limit lower=-3.14159 upper=3.14159 effort=0.0 velocity=0.0
- added joint Torso_UppperLeg11: type revolute, parent Torso, child UppperLeg11, origin xyz=-0.46488824294412573 0.18406227634233888 1 rpy=0 0 0, axis 0.36812455268467775 0.9297764858882515 0, limit lower=-3.14159 upper=3.14159 effort=0.0 velocity=0.0
- added joint Torso_UppperLeg12: type revolute, parent Torso, child UppperLeg12, origin xyz=-0.49605735065723894 0.06266661678215205 1 rpy=0 0 0, axis 0.1253332335643041 0.9921147013144779 0, limit lower=-3.14159 upper=3.14159 effort=0.0 velocity=0.0
- added joint Torso_UppperLeg13: type revolute, parent Torso, child UppperLeg13, origin xyz=-0.49605735065723894 -0.06266661678215214 1 rpy=0 0 0, axis 0.12533323356430429 0.9921147013144779 0, limit lower=-3.14159 upper=3.14159 effort=0.0 velocity=0.0
- added joint Torso_UppperLeg14: type revolute, parent Torso, child UppperLeg14, origin xyz=-0.46488824294412573 -0.18406227634233896 1 rpy=0 0 0, axis 0.3681245526846779 0.9297764858882515 0, limit lower=-3.14159 upper=3.14159 effort=0.0 velocity=0.0
- added joint Torso_UppperLeg15: type revolute, parent Torso, child UppperLeg15, origin xyz=-0.4045084971874737 -0.2938926261462365 1 rpy=0 0 0, axis 0.587785252292473 0.8090169943749475 0, limit lower=-3.14159 upper=3.14159 effort=0.0 velocity=0.0
- added joint Torso_UppperLeg16: type revolute, parent Torso, child UppperLeg16, origin xyz=-0.31871199487434476 -0.3852566213878947 1 rpy=0 0 0, axis 0.7705132427757894 0.6374239897486895 0, limit lower=-3.14159 upper=3.14159 effort=0.0 velocity=0.0
- added joint Torso_UppperLeg17: type revolute, parent Torso, child UppperLeg17, origin xyz=-0.21288964578253608 -0.4524135262330099 1 rpy=0 0 0, axis 0.9048270524660198 0.42577929156507216 0, limit lower=-3.14159 upper=3.14159 effort=0.0 velocity=0.0
- added joint Torso_UppperLeg18: type revolute, parent Torso, child UppperLeg18, origin xyz=-0.09369065729286231 -0.49114362536434436 1 rpy=0 0 0, axis 0.9822872507286887 0.18738131458572463 0, limit lower=-3.14159 upper=3.14159 effort=0.0 velocity=0.0
- added joint Torso_UppperLeg19: type revolute, parent Torso, child UppperLeg19, origin xyz=0.03139525976465686 -0.4990133642141358 1 rpy=0 0 0, axis 0.9980267284282716 0.06279051952931372 0, limit lower=-3.14159 upper=3.14159 effort=0.0 velocity=0.0
- added joint Torso_UppperLeg20: type revolute, parent Torso, child UppperLeg20, origin xyz=0.15450849718747361 -0.4755282581475768 1 rpy=0 0 0, axis 0.9510565162951536 0.30901699437494723 0, limit lower=-3.14159 upper=3.14159 effort=0.0 velocity=0.0
- added joint Torso_UppperLeg21: type revolute, parent Torso, child UppperLeg21, origin xyz=0.2679133974894984 -0.4221639627510075 1 rpy=0 0 0, axis 0.844327925502015 0.5358267949789968 0, limit lower=-3.14159 upper=3.14159 effort=0.0 velocity=0.0
- added joint Torso_UppperLeg22: type revolute, parent Torso, child UppperLeg22, origin xyz=0.36448431371070594 -0.34227355296434414 1 rpy=0 0 0, axis 0.6845471059286883 0.7289686274214119 0, limit lower=-3.14159 upper=3.14159 effort=0.0 velocity=0.0
- added joint Torso_UppperLeg23: type revolute, parent Torso, child UppperLeg23, origin xyz=0.4381533400219318 -0.24087683705085766 1 rpy=0 0 0, axis 0.4817536741017153 0.8763066800438636 0, limit lower=-3.14159 upper=3.14159 effort=0.0 velocity=0.0
- added joint Torso_UppperLeg24: type revolute, parent Torso, child UppperLeg24, origin xyz=0.4842915805643156 -0.12434494358242724 1 rpy=0 0 0, axis 0.2486898871648545 0.9685831611286312 0, limit lower=-3.14159 upper=3.14159 effort=0.0 velocity=0.0
- added joint Torso_UppperLeg4: type revolute, parent Torso, child UppperLeg4, origin xyz=0.2679133974894983 0.42216396275100754 1 rpy=0 0 0, axis 0.8443279255020151 0.5358267949789965 0, limit lower=-3.14159 upper=3.14159 effort=0.0 velocity=0.0
- added joint Torso_UppperLeg5: type revolute, parent Torso, child UppperLeg5, origin xyz=0.15450849718747373 0.47552825814757677 1 rpy=0 0 0, axis 0.9510565162951535 0.30901699437494745 0, limit lower=-3.14159 upper=3.14159 effort=0.0 velocity=0.0
- added joint Torso_UppperLeg6: type revolute, parent Torso, child UppperLeg6, origin xyz=0.03139525976465665 0.4990133642141358 1 rpy=0 0 0, axis 0.9980267284282716 0.0627905195293133 0, limit lower=-3.14159 upper=3.14159 effort=0.0 velocity=0.0
- added joint Torso_UppperLeg7: type revolute, parent Torso, child UppperLeg7, origin xyz=-0.0936906572928623 0.49114362536434436 1 rpy=0 0 0, axis 0.9822872507286887 0.1873813145857246 0, limit lower=-3.14159 upper=3.14159 effort=0.0 velocity=0.0
- added joint Torso_UppperLeg8: type revolute, parent Torso, child UppperLeg8, origin xyz=-0.21288964578253636 0.45241352623300973 1 rpy=0 0 0, axis 0.9048270524660195 0.4257792915650727 0, limit lower=-3.14159 upper=3.14159 effort=0.0 velocity=0.0
- added joint Torso_UppperLeg9: type revolute, parent Torso, child UppperLeg9, origin xyz=-0.3187119948743449 0.3852566213878946 1 rpy=0 0 0, axis 0.7705132427757893 0.6374239897486897 0, limit lower=-3.14159 upper=3.14159 effort=0.0 velocity=0.0
- added joint UppperLeg10_LowerLeg10: type revolute, parent UppperLeg10, child LowerLeg10, origin xyz=-0.8090169943749473 0.5877852522924732 0 rpy=0 0 0, axis 0.5877852522924732 0.8090169943749473 0, limit lower=-3.14159 upper=3.14159 effort=0.0 velocity=0.0
- added joint UppperLeg11_LowerLeg11: type revolute, parent UppperLeg11, child LowerLeg11, origin xyz=-0.9297764858882515 0.36812455268467775 0 rpy=0 0 0, axis 0.36812455268467775 0.9297764858882515 0, limit lower=-3.14159 upper=3.14159 effort=0.0 velocity=0.0
- added joint UppperLeg12_LowerLeg12: type revolute, parent UppperLeg12, child LowerLeg12, origin xyz=-0.9921147013144779 0.1253332335643041 0 rpy=0 0 0, axis 0.1253332335643041 0.9921147013144779 0, limit lower=-3.14159 upper=3.14159 effort=0.0 velocity=0.0
- added joint UppperLeg13_LowerLeg13: type revolute, parent UppperLeg13, child LowerLeg13, origin xyz=-0.9921147013144779 -0.12533323356430429 0 rpy=0 0 0, axis 0.12533323356430429 0.9921147013144779 0, limit lower=-3.14159 upper=3.14159 effort=0.0 velocity=0.0
- added joint UppperLeg14_LowerLeg14: type revolute, parent UppperLeg14, child LowerLeg14, origin xyz=-0.9297764858882515 -0.3681245526846779 0 rpy=0 0 0, axis 0.3681245526846779 0.9297764858882515 0, limit lower=-3.14159 upper=3.14159 effort=0.0 velocity=0.0
- added joint UppperLeg15_LowerLeg15: type revolute, parent UppperLeg15, child LowerLeg15, origin xyz=-0.8090169943749475 -0.587785252292473 0 rpy=0 0 0, axis 0.587785252292473 0.8090169943749475 0, limit lower=-3.14159 upper=3.14159 effort=0.0 velocity=0.0
- added joint UppperLeg16_LowerLeg16: type revolute, parent UppperLeg16, child LowerLeg16, origin xyz=-0.6374239897486895 -0.7705132427757894 0 rpy=0 0 0, axis 0.7705132427757894 0.6374239897486895 0, limit lower=-3.14159 upper=3.14159 effort=0.0 velocity=0.0
- added joint UppperLeg17_LowerLeg17: type revolute, parent UppperLeg17, child LowerLeg17, origin xyz=-0.42577929156507216 -0.9048270524660198 0 rpy=0 0 0, axis 0.9048270524660198 0.42577929156507216 0, limit lower=-3.14159 upper=3.14159 effort=0.0 velocity=0.0
- added joint UppperLeg18_LowerLeg18: type revolute, parent UppperLeg18, child LowerLeg18, origin xyz=-0.18738131458572463 -0.9822872507286887 0 rpy=0 0 0, axis 0.9822872507286887 0.18738131458572463 0, limit lower=-3.14159 upper=3.14159 effort=0.0 velocity=0.0
- added joint UppperLeg19_LowerLeg19: type revolute, parent UppperLeg19, child LowerLeg19, origin xyz=0.06279051952931372 -0.9980267284282716 0 rpy=0 0 0, axis 0.9980267284282716 0.06279051952931372 0, limit lower=-3.14159 upper=3.14159 effort=0.0 velocity=0.0
- added joint UppperLeg20_LowerLeg20: type revolute, parent UppperLeg20, child LowerLeg20, origin xyz=0.30901699437494723 -0.9510565162951536 0 rpy=0 0 0, axis 0.9510565162951536 0.30901699437494723 0, limit lower=-3.14159 upper=3.14159 effort=0.0 velocity=0.0
- added joint UppperLeg21_LowerLeg21: type revolute, parent UppperLeg21, child LowerLeg21, origin xyz=0.5358267949789968 -0.844327925502015 0 rpy=0 0 0, axis 0.844327925502015 0.5358267949789968 0, limit lower=-3.14159 upper=3.14159 effort=0.0 velocity=0.0
- added joint UppperLeg22_LowerLeg22: type revolute, parent UppperLeg22, child LowerLeg22, origin xyz=0.7289686274214119 -0.6845471059286883 0 rpy=0 0 0, axis 0.6845471059286883 0.7289686274214119 0, limit lower=-3.14159 upper=3.14159 effort=0.0 velocity=0.0
- added joint UppperLeg23_LowerLeg23: type revolute, parent UppperLeg23, child LowerLeg23, origin xyz=0.8763066800438636 -0.4817536741017153 0 rpy=0 0 0, axis 0.4817536741017153 0.8763066800438636 0, limit lower=-3.14159 upper=3.14159 effort=0.0 velocity=0.0
- added joint UppperLeg24_LowerLeg24: type revolute, parent UppperLeg24, child LowerLeg24, origin xyz=0.9685831611286312 -0.2486898871648545 0 rpy=0 0 0, axis 0.2486898871648545 0.9685831611286312 0, limit lower=-3.14159 upper=3.14159 effort=0.0 velocity=0.0
- added joint UppperLeg4_LowerLeg4: type revolute, parent UppperLeg4, child LowerLeg4, origin xyz=0.5358267949789965 0.8443279255020151 0 rpy=0 0 0, axis 0.8443279255020151 0.5358267949789965 0, limit lower=-3.14159 upper=3.14159 effort=0.0 velocity=0.0
- added joint UppperLeg5_LowerLeg5: type revolute, parent UppperLeg5, child LowerLeg5, origin xyz=0.30901699437494745 0.9510565162951535 0 rpy=0 0 0, axis 0.9510565162951535 0.30901699437494745 0, limit lower=-3.14159 upper=3.14159 effort=0.0 velocity=0.0
- added joint UppperLeg6_LowerLeg6: type revolute, parent UppperLeg6, child LowerLeg6, origin xyz=0.0627905195293133 0.9980267284282716 0 rpy=0 0 0, axis 0.9980267284282716 0.0627905195293133 0, limit lower=-3.14159 upper=3.14159 effort=0.0 velocity=0.0
- added joint UppperLeg7_LowerLeg7: type revolute, parent UppperLeg7, child LowerLeg7, origin xyz=-0.1873813145857246 0.9822872507286887 0 rpy=0 0 0, axis 0.9822872507286887 0.1873813145857246 0, limit lower=-3.14159 upper=3.14159 effort=0.0 velocity=0.0
- added joint UppperLeg8_LowerLeg8: type revolute, parent UppperLeg8, child LowerLeg8, origin xyz=-0.4257792915650727 0.9048270524660195 0 rpy=0 0 0, axis 0.9048270524660195 0.4257792915650727 0, limit lower=-3.14159 upper=3.14159 effort=0.0 velocity=0.0
- added joint UppperLeg9_LowerLeg9: type revolute, parent UppperLeg9, child LowerLeg9, origin xyz=-0.6374239897486897 0.7705132427757893 0 rpy=0 0 0, axis 0.7705132427757893 0.6374239897486897 0, limit lower=-3.14159 upper=3.14159 effort=0.0 velocity=0.0
- joint Torso_UppperLeg1: axis 1.0 6.123233995736766e-17 0 -> 0.2486898871648548 0.9685831611286311 0; origin xyz=3.061616997868383e-17 0.5 1 rpy=0 0 0 -> xyz=0.48429158056431554 0.1243449435824274 1 rpy=0 0 0
- joint Torso_UppperLeg2: axis 1.2246467991473532e-16 1.0 0 -> 0.4817536741017153 0.8763066800438636 0; origin xyz=-0.5 6.123233995736766e-17 1 rpy=0 0 0 -> xyz=0.4381533400219318 0.24087683705085766 1 rpy=0 0 0
- joint Torso_UppperLeg3: axis 1.0 1.8369701987210297e-16 0 -> 0.6845471059286887 0.7289686274214116 0; origin xyz=-9.184850993605148e-17 -0.5 1 rpy=0 0 0 -> xyz=0.3644843137107058 0.34227355296434436 1 rpy=0 0 0
- joint UppperLeg1_LowerLeg1: axis 1.0 6.123233995736766e-17 0 -> 0.2486898871648548 0.9685831611286311 0; origin xyz=6.123233995736766e-17 1.0 0 rpy=0 0 0 -> xyz=0.9685831611286311 0.2486898871648548 0 rpy=0 0 0
- joint UppperLeg2_LowerLeg2: axis 1.2246467991473532e-16 1.0 0 -> 0.4817536741017153 0.8763066800438636 0; origin xyz=-1.0 1.2246467991473532e-16 0 rpy=0 0 0 -> xyz=0.8763066800438636 0.4817536741017153 0 rpy=0 0 0
- joint UppperLeg3_LowerLeg3: axis 1.0 1.8369701987210297e-16 0 -> 0.6845471059286887 0.7289686274214116 0; origin xyz=-1.8369701987210297e-16 -1.0 0 rpy=0 0 0 -> xyz=0.7289686274214116 0.6845471059286887 0 rpy=0 0 0

Commit message: record the data

File: body.urdf (robot description, URDF)
Before this commit: robot robot, 51 links, 50 joints
Links:
- removed link LowerLeg10
- removed link LowerLeg11
- removed link LowerLeg12
- removed link LowerLeg13
- removed link LowerLeg14
- removed link LowerLeg15
- removed link LowerLeg16
- removed link LowerLeg17
- removed link LowerLeg18
- removed link LowerLeg19
- removed link LowerLeg20
- removed link LowerLeg21
- removed link LowerLeg22
- removed link LowerLeg23
- removed link LowerLeg24
- removed link LowerLeg4
- removed link LowerLeg5
- removed link LowerLeg6
- removed link LowerLeg7
- removed link LowerLeg8
- removed link LowerLeg9
- removed link UppperLeg10
- removed link UppperLeg11
- removed link UppperLeg12
- removed link UppperLeg13
- removed link UppperLeg14
- removed link UppperLeg15
- removed link UppperLeg16
- removed link UppperLeg17
- removed link UppperLeg18
- removed link UppperLeg19
- removed link UppperLeg20
- removed link UppperLeg21
- removed link UppperLeg22
- removed link UppperLeg23
- removed link UppperLeg24
- removed link UppperLeg4
- removed link UppperLeg5
- removed link UppperLeg6
- removed link UppperLeg7
- removed link UppperLeg8
- removed link UppperLeg9
Joints:
- removed joint Torso_UppperLeg10
- removed joint Torso_UppperLeg11
- removed joint Torso_UppperLeg12
- removed joint Torso_UppperLeg13
- removed joint Torso_UppperLeg14
- removed joint Torso_UppperLeg15
- removed joint Torso_UppperLeg16
- removed joint Torso_UppperLeg17
- removed joint Torso_UppperLeg18
- removed joint Torso_UppperLeg19
- removed joint Torso_UppperLeg20
- removed joint Torso_UppperLeg21
- removed joint Torso_UppperLeg22
- removed joint Torso_UppperLeg23
- removed joint Torso_UppperLeg24
- removed joint Torso_UppperLeg4
- removed joint Torso_UppperLeg5
- removed joint Torso_UppperLeg6
- removed joint Torso_UppperLeg7
- removed joint Torso_UppperLeg8
- removed joint Torso_UppperLeg9
- removed joint UppperLeg10_LowerLeg10
- removed joint UppperLeg11_LowerLeg11
- removed joint UppperLeg12_LowerLeg12
- removed joint UppperLeg13_LowerLeg13
- removed joint UppperLeg14_LowerLeg14
- removed joint UppperLeg15_LowerLeg15
- removed joint UppperLeg16_LowerLeg16
- removed joint UppperLeg17_LowerLeg17
- removed joint UppperLeg18_LowerLeg18
- removed joint UppperLeg19_LowerLeg19
- removed joint UppperLeg20_LowerLeg20
- removed joint UppperLeg21_LowerLeg21
- removed joint UppperLeg22_LowerLeg22
- removed joint UppperLeg23_LowerLeg23
- removed joint UppperLeg24_LowerLeg24
- removed joint UppperLeg4_LowerLeg4
- removed joint UppperLeg5_LowerLeg5
- removed joint UppperLeg6_LowerLeg6
- removed joint UppperLeg7_LowerLeg7
- removed joint UppperLeg8_LowerLeg8
- removed joint UppperLeg9_LowerLeg9
- joint Torso_UppperLeg1: axis 0.2486898871648548 0.9685831611286311 0 -> 1.0 6.123233995736766e-17 0; origin xyz=0.48429158056431554 0.1243449435824274 1 rpy=0 0 0 -> xyz=3.061616997868383e-17 0.5 1 rpy=0 0 0
- joint Torso_UppperLeg2: axis 0.4817536741017153 0.8763066800438636 0 -> 1.2246467991473532e-16 1.0 0; origin xyz=0.4381533400219318 0.24087683705085766 1 rpy=0 0 0 -> xyz=-0.5 6.123233995736766e-17 1 rpy=0 0 0
- joint Torso_UppperLeg3: axis 0.6845471059286887 0.7289686274214116 0 -> 1.0 1.8369701987210297e-16 0; origin xyz=0.3644843137107058 0.34227355296434436 1 rpy=0 0 0 -> xyz=-9.184850993605148e-17 -0.5 1 rpy=0 0 0
- joint UppperLeg1_LowerLeg1: axis 0.2486898871648548 0.9685831611286311 0 -> 1.0 6.123233995736766e-17 0; origin xyz=0.9685831611286311 0.2486898871648548 0 rpy=0 0 0 -> xyz=6.123233995736766e-17 1.0 0 rpy=0 0 0
- joint UppperLeg2_LowerLeg2: axis 0.4817536741017153 0.8763066800438636 0 -> 1.2246467991473532e-16 1.0 0; origin xyz=0.8763066800438636 0.4817536741017153 0 rpy=0 0 0 -> xyz=-1.0 1.2246467991473532e-16 0 rpy=0 0 0
- joint UppperLeg3_LowerLeg3: axis 0.6845471059286887 0.7289686274214116 0 -> 1.0 1.8369701987210297e-16 0; origin xyz=0.7289686274214116 0.6845471059286887 0 rpy=0 0 0 -> xyz=-1.8369701987210297e-16 -1.0 0 rpy=0 0 0

Commit message: the figure

File: body.urdf (robot description, URDF)
Before this commit: robot robot, 9 links, 8 joints
Links:
- added link LowerLeg4, mass 1; collision box size=0.2 0.2 1; visual box size=0.2 0.2 1
- added link LowerLeg5, mass 1; collision box size=0.2 0.2 1; visual box size=0.2 0.2 1
- added link UppperLeg4, mass 1; collision box size=1 0.2 0.2; visual box size=1 0.2 0.2
- added link UppperLeg5, mass 1; collision box size=1 0.2 0.2; visual box size=1 0.2 0.2
Joints:
- added joint Torso_UppperLeg4: type revolute, parent Torso, child UppperLeg4, origin xyz=-0.2500000000000002 -0.43301270189221924 1 rpy=0 0 0, axis 0.8660254037844385 0.5000000000000004 0, limit lower=-3.14159 upper=3.14159 effort=0.0 velocity=0.0
- added joint Torso_UppperLeg5: type revolute, parent Torso, child UppperLeg5, origin xyz=0.25000000000000006 -0.4330127018922193 1 rpy=0 0 0, axis 0.8660254037844386 0.5000000000000001 0, limit lower=-3.14159 upper=3.14159 effort=0.0 velocity=0.0
- added joint UppperLeg4_LowerLeg4: type revolute, parent UppperLeg4, child LowerLeg4, origin xyz=-0.5000000000000004 -0.8660254037844385 0 rpy=0 0 0, axis 0.8660254037844385 0.5000000000000004 0, limit lower=-3.14159 upper=3.14159 effort=0.0 velocity=0.0
- added joint UppperLeg5_LowerLeg5: type revolute, parent UppperLeg5, child LowerLeg5, origin xyz=0.5000000000000001 -0.8660254037844386 0 rpy=0 0 0, axis 0.8660254037844386 0.5000000000000001 0, limit lower=-3.14159 upper=3.14159 effort=0.0 velocity=0.0
- joint Torso_UppperLeg1: axis 1.0 6.123233995736766e-17 0 -> 0.8660254037844386 0.5000000000000001 0; origin xyz=3.061616997868383e-17 0.5 1 rpy=0 0 0 -> xyz=0.25000000000000006 0.4330127018922193 1 rpy=0 0 0
- joint Torso_UppperLeg2: axis 1.2246467991473532e-16 1.0 0 -> 0.8660254037844387 0.4999999999999998 0; origin xyz=-0.5 6.123233995736766e-17 1 rpy=0 0 0 -> xyz=-0.2499999999999999 0.43301270189221935 1 rpy=0 0 0
- joint Torso_UppperLeg3: axis 1.0 1.8369701987210297e-16 0 -> 1.2246467991473532e-16 1.0 0; origin xyz=-9.184850993605148e-17 -0.5 1 rpy=0 0 0 -> xyz=-0.5 6.123233995736766e-17 1 rpy=0 0 0
- joint UppperLeg1_LowerLeg1: axis 1.0 6.123233995736766e-17 0 -> 0.8660254037844386 0.5000000000000001 0; origin xyz=6.123233995736766e-17 1.0 0 rpy=0 0 0 -> xyz=0.5000000000000001 0.8660254037844386 0 rpy=0 0 0
- joint UppperLeg2_LowerLeg2: axis 1.2246467991473532e-16 1.0 0 -> 0.8660254037844387 0.4999999999999998 0; origin xyz=-1.0 1.2246467991473532e-16 0 rpy=0 0 0 -> xyz=-0.4999999999999998 0.8660254037844387 0 rpy=0 0 0
- joint UppperLeg3_LowerLeg3: axis 1.0 1.8369701987210297e-16 0 -> 1.2246467991473532e-16 1.0 0; origin xyz=-1.8369701987210297e-16 -1.0 0 rpy=0 0 0 -> xyz=-1.0 1.2246467991473532e-16 0 rpy=0 0 0
