Commit message: all done a/b tesing

File: body.urdf (robot description, URDF)
Before this commit: robot robot, 13 links, 12 joints
Links:
- removed link LowerLeg4
- removed link LowerLeg5
- removed link UppperLeg4
- removed link UppperLeg5
Joints:
- removed joint Torso_UppperLeg4
- removed joint Torso_UppperLeg5
- removed joint UppperLeg4_LowerLeg4
- removed joint UppperLeg5_LowerLeg5
- joint Torso_UppperLeg1: axis 0.8660254037844386 0.5000000000000001 0 -> 1.0 6.123233995736766e-17 0; origin xyz=0.25000000000000006 0.4330127018922193 1 rpy=0 0 0 -> xyz=3.061616997868383e-17 0.5 1 rpy=0 0 0
- joint Torso_UppperLeg2: axis 0.8660254037844387 0.4999999999999998 0 -> 1.2246467991473532e-16 1.0 0; origin xyz=-0.2499999999999999 0.43301270189221935 1 rpy=0 0 0 -> xyz=-0.5 6.123233995736766e-17 1 rpy=0 0 0
- joint Torso_UppperLeg3: axis 1.2246467991473532e-16 1.0 0 -> 1.0 1.8369701987210297e-16 0; origin xyz=-0.5 6.123233995736766e-17 1 rpy=0 0 0 -> xyz=-9.184850993605148e-17 -0.5 1 rpy=0 0 0
- joint UppperLeg1_LowerLeg1: axis 0.8660254037844386 0.5000000000000001 0 -> 1.0 6.123233995736766e-17 0; origin xyz=0.5000000000000001 0.8660254037844386 0 rpy=0 0 0 -> xyz=6.123233995736766e-17 1.0 0 rpy=0 0 0
- joint UppperLeg2_LowerLeg2: axis 0.8660254037844387 0.4999999999999998 0 -> 1.2246467991473532e-16 1.0 0; origin xyz=-0.4999999999999998 0.8660254037844387 0 rpy=0 0 0 -> xyz=-1.0 1.2246467991473532e-16 0 rpy=0 0 0
- joint UppperLeg3_LowerLeg3: axis 1.2246467991473532e-16 1.0 0 -> 1.0 1.8369701987210297e-16 0; origin xyz=-1.0 1.2246467991473532e-16 0 rpy=0 0 0 -> xyz=-1.8369701987210297e-16 -1.0 0 rpy=0 0 0
